Commit message: stl修正

File: ROS/harvest-studio/urdf/harvest-studio.urdf (robot description, URDF)
Before this commit: robot harvest-studio, 2 links, 1 joints
Links:
- link camera-link: mass 2.78889228470616 -> 2.7889
- link harest-base: mass 10.2467447687249 -> 10.247

Commit message: stl修正

File: ROS/harvest-studio/urdf/harvest-studio.urdf (robot description, URDF)
Before this commit: robot harvest-studio, 2 links, 1 joints
Links:
- link camera-link: mass 2.7889 -> 2.78889236681532
- link harest-base: mass 10.247 -> 10.2530883442845

Commit message: tf修正

File: ROS/harvest-studio/urdf/harvest-studio.urdf (robot description, URDF)
Before this commit: robot harvest-studio, 2 links, 1 joints
Links:
- removed link camera-link
- removed link harest-base
- added link camera_link, mass 2.78889236681529; collision mesh filename=package://harvest-studio/meshes/camera_link.STL; visual mesh filename=package://harvest-studio/meshes/camera_link.STL
- added link stand_base, mass 0.109449715271813; collision mesh filename=package://harvest-studio/meshes/stand_base.STL; visual mesh filename=package://harvest-studio/meshes/stand_base.STL
Joints:
- joint camera_joint: child camera-link -> camera_link; limit lower=-0.5 upper=0.5 effort=0 velocity=0 -> lower=0 upper=0 effort=0 velocity=0; origin xyz=-0.55495 -0.675 0.80244 rpy=-0.20407 0 3.1416 -> xyz=0.00085 0.465 0.98 rpy=0 0 -3.1416; parent harest-base -> stand_base

Commit message: tf修正

File: ROS/harvest-studio/urdf/harvest-studio.urdf (robot description, URDF)
Before this commit: robot harvest-studio, 2 links, 1 joints
Links:
- link stand_base: mass 0.109449715271813 -> 10.2530883442845
Joints:
- joint camera_joint: limit lower=0 upper=0 effort=0 velocity=0 -> lower=-0.5 upper=0.5 effort=0 velocity=0; type revolute -> fixed

Commit message: change joint mode

File: ROS/harvest-studio/urdf/harvest-studio.urdf (robot description, URDF)
Before this commit: robot harvest-studio, 2 links, 1 joints
Joints:
- joint camera_joint: type fixed -> revolute
